Commit message: add rgbd and add mujoco

File: urdf/ur.ros2_control.xacro (robot description, xacro)
@@ -18,5 +18,7 @@
     script_sender_port:=50002
     reverse_ip:=0.0.0.0
-    script_command_port:=50004">
+    script_command_port:=50004
+    mujoco_model
+    sim_mujoco">
     <ros2_control name="${name}" type="system">
       <hardware>
@@ -27,4 +29,8 @@
           <plugin>ign_ros2_control/IgnitionSystem</plugin>
         </xacro:if>
+        <xacro:if value="${sim_mujoco}">
+          <plugin>cartesian_controller_simulation/Simulator</plugin>
+          <param name="mujoco_model">${mujoco_model}</param>
+        </xacro:if>
         <xacro:if value="${use_fake_hardware}">
           <plugin>mock_components/GenericSystem</plugin>
@@ -32,5 +38,5 @@
           <param name="state_following_offset">0.0</param>
         </xacro:if>
-        <xacro:unless value="${use_fake_hardware or sim_gazebo or sim_ignition}">
+        <xacro:unless value="${use_fake_hardware or sim_gazebo or sim_ignition or sim_mujoco}">
           <plugin>ur_robot_driver/URPositionHardwareInterface</plugin>
           <param name="robot_ip">${robot_ip}</param>
@@ -155,5 +161,5 @@
         <state_interface name="effort"/>
       </joint>
-      <xacro:unless value="${sim_gazebo or sim_ignition}">
+      <xacro:unless value="${sim_gazebo or sim_ignition or sim_mujoco}">
         <sensor name="tcp_fts_sensor">
           <state_interface name="force.x"/>

File: urdf/ur.urdf.xacro (robot description, xacro)
@@ -9,5 +9,6 @@
    <xacro:include filename="$(find rbs_simulation)/table/table.xacro"/>
    <xacro:include filename="$(find ur_description)/urdf/plane_macro.xacro"/>
-   <xacro:include filename="$(find ur_description)/urdf/camera.xacro"/>
+   <xacro:include filename="$(find ur_description)/urdf/key_frames.xacro"/>
+   <xacro:include filename="$(find ur_description)/urdf/sensors.xacro"/>
    <!-- possible 'ur_type' values: ur3, ur3e, ur5, ur5e, ur10, ur10e, ur16e -->
    <!-- the default value should raise an error in case this was called without defining the type -->
@@ -47,5 +48,7 @@
    <xacro:arg name="sim_gazebo" default="false" />
    <xacro:arg name="sim_ignition" default="false" />
+   <xacro:arg name="sim_mujoco" default="false" />
    <xacro:arg name="simulation_controllers" default="" />
+   <xacro:arg name="mujoco_model" default=""/>
    <!-- initial position for simulations (Fake Hardware, Gazebo, Ignition) -->
    <xacro:arg name="initial_positions_file" default="$(find ur_description)/config/initial_positions.yaml"/>
@@ -71,4 +74,6 @@
      sim_gazebo="$(arg sim_gazebo)"
      sim_ignition="$(arg sim_ignition)"
+     sim_mujoco="$(arg sim_mujoco)"
+     mujoco_model="$(arg mujoco_model)"
      headless_mode="$(arg headless_mode)"
      initial_positions="${xacro.load_yaml(initial_positions_file)}"
@@ -94,5 +99,8 @@
     <origin xyz="0.0 1.0 1.0" rpy="0.0 0.0 0.0"/>
    </xacro:camera>
-   <xacro:plane parent="world">
+   <xacro:camera parent="base_link">
+    <origin xyz="0.0 1.0 1.0" rpy="0.0 0.0 0.0"/>
+   </xacro:camera>
+   <!-- <xacro:plane parent="world">
         <origin xyz="0 0 -0.001" rpy="0 0 0"/>
    </xacro:plane>
@@ -102,7 +110,7 @@
     <xacro:table parent="world">
         <origin xyz="-0.75 0.0 0.2" rpy="0.0 0.0 0.0"/>
-    </xacro:table>
+    </xacro:table> -->
    <xacro:if value="$(arg with_gripper)">
-        <xacro:robotiq_gripper parent="tool0" sim="true" prefix="">
+        <xacro:robotiq_gripper parent="tool0" sim="true" prefix="" sim_mujoco="$(arg sim_mujoco)" mujoco_model="$(arg mujoco_model)">
             <origin xyz="0 0 0" rpy="0 0 0" />
         </xacro:robotiq_gripper>
@@ -120,4 +128,7 @@
   <xacro:if value="$(arg sim_ignition)">
     <!-- Gazebo plugins -->
+    <xacro:rgbd parent="tool0" prefix="">
+            <origin xyz="0 -0.05 0.07" rpy="1.57 -1.57 0" />
+    </xacro:rgbd>
     <gazebo reference="world">
     </gazebo>

File: urdf/ur_macro.xacro (robot description, xacro)
@@ -61,4 +61,5 @@
     sim_gazebo:=false
     sim_ignition:=false
+    sim_mujoco:=false
     headless_mode:=false
     initial_positions:=${dict(shoulder_pan_joint=0.0,shoulder_lift_joint=-1.57,elbow_joint=0.0,wrist_1_joint=-1.57,wrist_2_joint=0.0,wrist_3_joint=0.0)}
@@ -79,5 +80,6 @@
     script_sender_port:=50002
     reverse_ip:=0.0.0.0
-    script_command_port:=50004">
+    script_command_port:=50004
+    mujoco_model">
     <!-- Load configuration data from the provided .yaml files -->
     <xacro:read_model_data
@@ -98,4 +100,5 @@
       sim_gazebo="${sim_gazebo}"
       sim_ignition="${sim_ignition}"
+      sim_mujoco="${sim_mujoco}"
       script_filename="${script_filename}"
       output_recipe_filename="${output_recipe_filename}"
@@ -117,4 +120,5 @@
       reverse_ip="${reverse_ip}"
       script_command_port="${script_command_port}"
+      mujoco_model="${mujoco_model}"
       />
     <!-- Add URDF transmission elements (for ros_control) -->

Commit message: add cartesian controller params and fix errors

File: urdf/ur.ros2_control.xacro (robot description, xacro)
@@ -1,4 +1,5 @@
 <?xml version="1.0"?>
 <robot xmlns:xacro="http://www.ros.org/wiki/xacro">
+<xacro:include filename="$(find ur_description)/urdf/inc/joint_interface.xacro"/>
   <xacro:macro name="ur_ros2_control" params="
     name
@@ -35,5 +36,5 @@
         <xacro:if value="${use_fake_hardware}">
           <plugin>mock_components/GenericSystem</plugin>
-          <param name="fake_sensor_commands">${fake_sensor_commands}</param>
+          <param name="mock_sensor_commands">${fake_sensor_commands}</param>
           <param name="state_following_offset">0.0</param>
         </xacro:if>
@@ -65,100 +66,10 @@
         </xacro:unless>
       </hardware>
-      <joint name="${prefix}shoulder_pan_joint">
-        <command_interface name="position">
-          <param name="min">{-2*pi}</param>
-          <param name="max">{2*pi}</param>
-        </command_interface>
-        <command_interface name="velocity">
-          <param name="min">-3.15</param>
-          <param name="max">3.15</param>
-        </command_interface>
-        <state_interface name="position">
-          <!-- initial position for the FakeSystem and simulation -->
-          <param name="initial_value">${initial_positions['shoulder_pan_joint']}</param>
-        </state_interface>
-        <state_interface name="velocity"/>
-        <state_interface name="effort"/>
-      </joint>
-      <joint name="${prefix}shoulder_lift_joint">
-        <command_interface name="position">
-          <param name="min">{-2*pi}</param>
-          <param name="max">{2*pi}</param>
-        </command_interface>
-        <command_interface name="velocity">
-          <param name="min">-3.15</param>
-          <param name="max">3.15</param>
-        </command_interface>
-        <state_interface name="position">
-          <!-- initial position for the FakeSystem and simulation -->
-          <param name="initial_value">${initial_positions['shoulder_lift_joint']}</param>
-        </state_interface>
-        <state_interface name="velocity"/>
-        <state_interface name="effort"/>
-      </joint>
-      <joint name="${prefix}elbow_joint">
-        <command_interface name="position">
-          <param name="min">{-pi}</param>
-          <param name="max">{pi}</param>
-        </command_interface>
-        <command_interface name="velocity">
-          <param name="min">-3.15</param>
-          <param name="max">3.15</param>
-        </command_interface>
-        <state_interface name="position">
-          <!-- initial position for the FakeSystem and simulation -->
-          <param name="initial_value">${initial_positions['elbow_joint']}</param>
-        </state_interface>
-        <state_interface name="velocity"/>
-        <state_interface name="effort"/>
-      </joint>
-      <joint name="${prefix}wrist_1_joint">
-        <command_interface name="position">
-          <param name="min">{-2*pi}</param>
-          <param name="max">{2*pi}</param>
-        </command_interface>
-        <command_interface name="velocity">
-          <param name="min">-3.2</param>
-          <param name="max">3.2</param>
-        </command_interface>
-        <state_interface name="position">
-          <!-- initial position for the FakeSystem and simulation -->
-          <param name="initial_value">${initial_positions['wrist_1_joint']}</param>
-        </state_interface>
-        <state_interface name="velocity"/>
-        <state_interface name="effort"/>
-      </joint>
-      <joint name="${prefix}wrist_2_joint">
-        <command_interface name="position">
-          <param name="min">{-2*pi}</param>
-          <param name="max">{2*pi}</param>
-        </command_interface>
-        <command_interface name="velocity">
-          <param name="min">-3.2</param>
-          <param name="max">3.2</param>
-        </command_interface>
-        <state_interface name="position">
-          <!-- initial position for the FakeSystem and simulation -->
-          <param name="initial_value">${initial_positions['wrist_2_joint']}</param>
-        </state_interface>
-        <state_interface name="velocity"/>
-        <state_interface name="effort"/>
-      </joint>
-      <joint name="${prefix}wrist_3_joint">
-        <command_interface name="position">
-          <param name="min">{-2*pi}</param>
-          <param name="max">{2*pi}</param>
-        </command_interface>
-        <command_interface name="velocity">
-          <param name="min">-3.2</param>
-          <param name="max">3.2</param>
-        </command_interface>
-        <state_interface name="position">
-          <!-- initial position for the FakeSystem and simulation -->
-          <param name="initial_value">${initial_positions['wrist_3_joint']}</param>
-        </state_interface>
-        <state_interface name="velocity"/>
-        <state_interface name="effort"/>
-      </joint>
+        <xacro:joint_interface name="${prefix}shoulder_pan_joint"   p="1000"    d="0.5" />
+        <xacro:joint_interface name="${prefix}shoulder_lift_joint"  p="1000"    d="0.5" />
+        <xacro:joint_interface name="${prefix}elbow_joint"          p="500"     d="0.5" />
+        <xacro:joint_interface name="${prefix}wrist_1_joint"        p="100"     d="0.5" />
+        <xacro:joint_interface name="${prefix}wrist_2_joint"        p="10"      d="0.5" />
+        <xacro:joint_interface name="${prefix}wrist_3_joint"        p="10"      d="0.5" />
       <xacro:unless value="${sim_gazebo or sim_ignition or sim_mujoco}">
         <sensor name="tcp_fts_sensor">

File: urdf/ur.urdf.xacro (robot description, xacro)
@@ -96,19 +96,7 @@
      <origin xyz="0 0 0" rpy="0 0 0" />          <!-- position robot in the world -->
    </xacro:ur_robot>
-   <xacro:camera parent="base_link">
+   <!-- <xacro:camera parent="base_link">
     <origin xyz="0.0 1.0 1.0" rpy="0.0 0.0 0.0"/>
-   </xacro:camera>
-   <xacro:camera parent="base_link">
-    <origin xyz="0.0 1.0 1.0" rpy="0.0 0.0 0.0"/>
-   </xacro:camera>
-   <!-- <xacro:plane parent="world">
-        <origin xyz="0 0 -0.001" rpy="0 0 0"/>
-   </xacro:plane>
-    <xacro:rack parent="world">
-        <origin xyz="0.0 0.7 0.0" rpy="0.0 0.0 0.0"/>
-    </xacro:rack>
-    <xacro:table parent="world">
-        <origin xyz="-0.75 0.0 0.2" rpy="0.0 0.0 0.0"/>
-    </xacro:table> -->
+   </xacro:camera> -->
    <xacro:if value="$(arg with_gripper)">
         <xacro:robotiq_gripper parent="tool0" sim="true" prefix="" sim_mujoco="$(arg sim_mujoco)" mujoco_model="$(arg mujoco_model)">
