Commit message: update poses and update rgbd_camera macro

File: urdf/key_frames.xacro (robot description, xacro)
@@ -10,20 +10,20 @@
   </xacro:macro>
 <xacro:key_frame name="box1_place">
-    <origin xyz="-0.45 -0.055 0.46" rpy="-3.1415927 0.0 0.0"/>
+    <origin xyz="-0.45 -0.055 0.025" rpy="-3.1415927 0.0 0.0"/>
 </xacro:key_frame>
 <xacro:key_frame name="box2_place">
-    <origin xyz="-0.45 0.0 0.46" rpy="-3.1415927 0.0 0.0"/>
+    <origin xyz="-0.45 0.0 0.025" rpy="-3.1415927 0.0 0.0"/>
 </xacro:key_frame>
 <xacro:key_frame name="box3_place">
-    <origin xyz="-0.45 0.055 0.46" rpy="-3.1415927 0.0 0.0"/>
+    <origin xyz="-0.45 0.055 0.025" rpy="-3.1415927 0.0 0.0"/>
 </xacro:key_frame>
 <xacro:key_frame name="box4_place">
-    <origin xyz="-0.45 0.0275 0.49" rpy="-3.1415927 0.0 0.0"/>
+    <origin xyz="-0.45 0.0275 0.055" rpy="-3.1415927 0.0 0.0"/>
 </xacro:key_frame>
 <xacro:key_frame name="box5_place">
-    <origin xyz="-0.45 -0.0275 0.49" rpy="-3.1415927 0.0 0.0"/>
+    <origin xyz="-0.45 -0.0275 0.055" rpy="-3.1415927 0.0 0.0"/>
 </xacro:key_frame>
 <xacro:key_frame name="box6_place">
-    <origin xyz="-0.45 0 0.56" rpy="-3.1415927 0.0 0.0"/>
+    <origin xyz="-0.45 0 0.125" rpy="-3.1415927 0.0 0.0"/>
 </xacro:key_frame>
 </robot>

File: urdf/sensors.xacro (robot description, xacro)
@@ -2,9 +2,9 @@
 <robot xmlns:xacro="http://www.ros.org/wiki/xacro" name="rack">
     <xacro:macro name="rgbd" params="*origin parent prefix">
-        <link name="rgbd_camera">
+        <link name="${prefix}rgbd_camera">
             <inertial>
                 <origin xyz="0.0 0.0 0.0" rpy="0.0 0.0 0.0"/>
                 <mass value="0.1"/>
-                <inertia ixx="0.0" ixy="0.0" ixz="0.0" iyy="0.0" iyz="0.0" izz="0.0"/>
+                <inertia ixx="0.000166667" ixy="0.0" ixz="0.0" iyy="0.000166667" iyz="0.0" izz="0.000166667"/>
             </inertial>
             <visual name="">
@@ -25,6 +25,6 @@
             </collision>
         </link>
-        <gazebo reference = "rgbd_camera">
-            <sensor name="rgbd_camera" type="rgbd_camera">
+        <gazebo reference = "${prefix}rgbd_camera">
+            <sensor name="${prefix}rgbd_camera" type="rgbd_camera">
                 <camera>
                     <horizontal_fov>1.047</horizontal_fov>
@@ -41,11 +41,11 @@
                 <update_rate>30</update_rate>
                 <visualize>true</visualize>
-                <topic>rgbd_camera</topic>
+                <topic>${prefix}rgbd_camera</topic>
                 <enable_metrics>true</enable_metrics>
             </sensor>
         </gazebo>
-        <joint name="plane_base_joint" type="fixed">
+        <joint name="${prefix}rgbd_camera_to_parent" type="fixed">
             <parent link="${parent}" />
-            <child link="rgbd_camera" />
+            <child link="${prefix}rgbd_camera" />
             <xacro:insert_block name="origin" />
         </joint>

File: urdf/ur.urdf.xacro (robot description, xacro)
@@ -111,6 +111,10 @@
   <xacro:if value="$(arg sim_gazebo)">
     <!-- Gazebo plugins -->
-    <xacro:rgbd parent="tool0" prefix="">
+    <xacro:rgbd parent="tool0" prefix="inner_">
             <origin xyz="0 -0.05 0.07" rpy="1.57 -1.57 0" />
+    </xacro:rgbd>
+    <!-- -2.0 -0.55 1.44 0 0.44 0.44 -->
+    <xacro:rgbd parent="world" prefix="outer_">
+            <origin xyz="-2.0 -0.55 1.44" rpy="0 0.44 0.44" />
     </xacro:rgbd>
     <gazebo reference="world">
