Commit message: add ft-sensor

File: urdf/sensors.xacro (robot description, xacro)
@@ -51,3 +51,33 @@
         </joint>
     </xacro:macro>
+    <xacro:macro name="rbs_fts" params="name prefix link">
+    <ros2_control name="${name}" type="sensor">
+      <hardware>
+          <plugin>ign_ros2_control/IgnitionFts</plugin>
+      </hardware>
+      <sensor name="${prefix}${name}">
+        <state_interface name="force.x"/>
+        <state_interface name="force.y"/>
+        <state_interface name="force.z"/>
+        <state_interface name="torque.x"/>
+        <state_interface name="torque.y"/>
+        <state_interface name="torque.z"/>
+      </sensor>
+    </ros2_control>
+    <gazebo>
+        <plugin filename="ignition-gazebo-forcetorque-system" name="ignition::gazebo::systems::ForceTorque"/>
+    </gazebo>
+    <gazebo reference="${prefix}${link}">
+        <sensor name="${prefix}${name}" type="force_torque">
+          <always_on>1</always_on>
+          <update_rate>10.0</update_rate>
+          <visualize>true</visualize>
+          <topic>ft_data</topic>
+          <force_torque>
+            <frame>sensor</frame>
+            <measure_direction>child_to_parent</measure_direction>
+          </force_torque>
+        </sensor>
+      </gazebo>
+  </xacro:macro>
 </robot>

File: urdf/ur.ros2_control.xacro (robot description, xacro)
@@ -68,14 +68,4 @@
         <xacro:joint_interface name="${prefix}wrist_2_joint"        p="10"      d="0.5" />
         <xacro:joint_interface name="${prefix}wrist_3_joint"        p="10"      d="0.5" />
-        <xacro:if value="${sim_gazebo}">
-            <sensor name="ft_sensor">
-                <state_interface name="force.x"/>
-                <state_interface name="force.y"/>
-                <state_interface name="force.z"/>
-                <state_interface name="torque.x"/>
-                <state_interface name="torque.y"/>
-                <state_interface name="torque.z"/>
-              </sensor>
-        </xacro:if>
       <xacro:unless value="${sim_gazebo or sim_mujoco}">
         <sensor name="tcp_fts_sensor">

File: urdf/ur.urdf.xacro (robot description, xacro)
@@ -121,9 +121,6 @@
         <controller_manager_node_name>$(arg prefix)controller_manager</controller_manager_node_name>
       </plugin>
-      <plugin
-      filename="ignition-gazebo-forcetorque-system"
-      name="ignition::gazebo::systems::ForceTorque">
-    </plugin>
     </gazebo>
+    <xacro:rbs_fts name = "ft_sensor" prefix="" link="ft_frame"/>
   </xacro:if>
 </robot>

File: urdf/ur_macro.xacro (robot description, xacro)
@@ -381,16 +381,4 @@
       <child link="${prefix}tool0"/>
     </joint>
-    <gazebo reference="${prefix}tool0">
-        <sensor name="ft_sensor" type="force_torque">
-          <always_on>1</always_on>
-          <update_rate>10.0</update_rate>
-          <visualize>true</visualize>
-          <topic>force_and_torque</topic>
-          <force_torque>
-            <frame>sensor</frame>
-            <measure_direction>child_to_parent</measure_direction>
-          </force_torque>
-        </sensor>
-      </gazebo>
   </xacro:macro>
 </robot>

Commit message: update description for real setup

File: urdf/sensors.xacro (robot description, xacro)
@@ -45,5 +45,5 @@
             </sensor>
         </gazebo>
-        <joint name="${prefix}rgbd_camera_to_parent" type="fixed">
+        <joint name="${prefix}rgbd_camera_joint" type="fixed">
             <parent link="${parent}" />
             <child link="${prefix}rgbd_camera" />

File: urdf/ur.urdf.xacro (robot description, xacro)
@@ -5,5 +5,5 @@
    <!-- import main macro -->
    <xacro:include filename="$(find ur_description)/urdf/ur_macro.xacro"/>
-   <xacro:include filename="$(find robotiq_description)/urdf/robotiq_gripper_macro.urdf.xacro" />
+   <xacro:include filename="$(find rbs_schunk_egp_n_n_b)/urdf/schunk_gripper_macro.xacro"/>
    <xacro:include filename="$(find rbs_simulation)/rack/rack.xacro"/>
    <xacro:include filename="$(find rbs_simulation)/table/table.xacro"/>
@@ -98,14 +98,7 @@
    </xacro:camera> -->
    <xacro:if value="$(arg with_gripper)">
-        <xacro:robotiq_gripper
-        parent="tool0"
-        sim="true"
-        prefix=""
-        sim_mujoco="$(arg sim_mujoco)"
-        mujoco_model="$(arg mujoco_model)"
-        sim_gazebo="$(arg sim_gazebo)"
-        use_fake_hardware="$(arg sim_fake)">
-            <origin xyz="0 0 0" rpy="0 0 0" />
-        </xacro:robotiq_gripper>
+        <xacro:schunk_gripper prefix="schunk" parent="tool0" sim_name="gazebo">
+          <origin xyz="0.0 0.0 0.0" rpy="0.0 0.0 0.0"/>
+        </xacro:schunk_gripper>
    </xacro:if>
   <xacro:if value="$(arg sim_gazebo)">
